Commit message: working

File: cora_description/urdf/cora.urdf.xacro (robot description, xacro)
@@ -1,13 +1,15 @@
 <?xml version="1.0"?>
 <robot xmlns:xacro="http://ros.org/wiki/xacro" name="cora">
+  <xacro:arg name="namespace" default="cora"/>
+  <xacro:property name="namespace" value="$(arg namespace)" scope="global" />
   <link name="base_link">
   </link>
-  <joint name="dummy_joint" type="fixed">
+  <joint name="${namespace}/base_link" type="fixed">
     <parent link="base_link"/>
-    <child link="dummy_link"/>
+    <child link="${namespace}/base_link"/>
     <!-- Adjust the visual/collision to match water height -->
     <origin xyz="0 0 1" rpy="0 0 0"/>
   </joint>
-  <link name="dummy_link">
+  <link name="${namespace}/base_link">
     <visual>
       <origin xyz="0 0 0" rpy="0 0 0" />
@@ -41,6 +43,6 @@
 a circle segment. The value for the draft is consistent specifications of similar vessels.  Moments of inertia are based on an effective cylindrical model-->
     <inertial>
-       <mass value="33000.0"/>
-       <inertia ixx="20700.0" ixy="0.0" ixz="0.0" iyy="420000.0" iyz="0.0" izz="420000.0"/>
+      <mass value="33000.0"/>
+      <inertia ixx="20700.0" ixy="0.0" ixz="0.0" iyy="420000.0" iyz="0.0" izz="420000.0"/>
     </inertial>
   </link>

File: cora_description/urdf/thrusters.xacro (robot description, xacro)
@@ -41,5 +41,5 @@
     <axis xyz="0 0 1"/>
     <origin rpy="0 0 0" xyz="-6.103 0.911 0.016"/>
-    <parent link="base_link"/>
+    <parent link="${namespace}/base_link"/>
     <child link="left_engine_link"/>
     <limit lower="${-pi}" upper="${pi}" effort="10" velocity="10"/>
@@ -93,5 +93,5 @@
     <axis xyz="0 0 1"/>
     <origin rpy="0 0 0" xyz="-6.103 -0.911 0.016"/>
-    <parent link="base_link"/>
+    <parent link="${namespace}/base_link"/>
     <child link="right_engine_link"/>
     <limit lower="${-pi}" upper="${pi}" effort="10" velocity="10"/>
